File: PCB_Temperature_sensor_V1/Temperature_sensor.kicad_sch (KiCad schematic)
At the start: 35 parts, among them IC1 TC7660, J1 BAT_GND, J2 BAT_3.7V, SW1 SW_Push, SW2 SW_Push, SW3 SW_Push, U1 TP4056, U2 ESP32-S3-ZERO, U3 LM35-LP, U4 DM-OLED096-636

Commit message: final
Other:
- moved on the sheet: C1, C2, C3, C4, C8, C9, D1, D2, H1, H2, H3, H4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
