File: PCB_Temperature_sensor_V1/Temperature_sensor.kicad_pcb (KiCad board)
At the start: 2 copper layers, 88.4 x 56.5 mm, 41 parts, among them SW1 SW_Push, SW2 SW_Push, SW3 SW_Push

Commit message: Final
Other:
- board size 88.4 x 56.5 mm -> 41.1 x 55.2 mm
Changed lines of the file:
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@@
 		)
-	)
-	(gr_circle
-		(center 112.26 107.03)
-		(end 114.198376 107.03)
-		(stroke
-			(width 0.5)
-			(type default)
-		)
-		(fill none)
-		(layer "Edge.Cuts")
-	)
-	(gr_circle
-		(center 78.64 59.39)
-		(end 80.578376 59.39)
-		(stroke
-			(width 0.5)
-			(type default)
-		)
-		(fill none)
-		(layer "Edge.Cuts")
-	)
-	(gr_circle
-		(center 79.01 107.08)
-		(end 80.948376 107.08)
-		(stroke
-			(width 0.5)
-			(type default)
-		)
-		(fill none)
-		(layer "Edge.Cuts")
-	)
-	(gr_circle
-		(center 112.368375 59.28)
-		(end 114.306751 59.28)
-		(stroke
-			(width 0.5)
-			(type default)
-		)
-		(fill none)
-		(layer "Edge.Cuts")
 	)
 	(gr_rect
@@
 			(type solid)
 		)
-		(fill none)
-		(layer "Edge.Cuts")
-	)
-	(gr_poly
-		(pts
-			(xy 74.963375 55.535) (xy 74.963375 110.765) (xy 85.688375 110.74) (xy 85.948375 84.66) (xy 106.008375 84.62)
-			(xy 106.058375 110.77) (xy 116.093375 110.765) (xy 116.093375 55.535)
-		)
-		(stroke
-			(width 0.5)
-			(type solid)
-		)
