File: PCB_Temperature_sensor_V2/PCB_Temperature_sensor_V2.kicad_sch (KiCad schematic)
At the start: 11 parts, among them U1 LM35-LP, U2 LM358, U3 LM358

Commit message: B2
Parts:
- removed R2, R3: R, Resistor_THT:R_Axial_DIN0207_L6.3mm_D2.5mm_P7.62mm_Horizontal, symbol Device:R
- removed U1: LM35-LP, Package_TO_SOT_THT:TO-92_Inline, symbol Sensor_Temperature:LM35-LP
- added J1: Conn_01x04_Pin, Connector_PinHeader_2.54mm:PinHeader_1x04_P2.54mm_Vertical, symbol Connector:Conn_01x04_Pin
- added J2, J3: Conn_01x02_Pin, Connector_PinHeader_2.54mm:PinHeader_1x02_P2.54mm_Vertical, symbol Connector:Conn_01x02_Pin
- added RV1, RV2: R_Potentiometer, Potentiometer_THT:Potentiometer_Piher_PT-10-V10_Vertical, symbol Device:R_Potentiometer
- R1, R4, R5, R6, R7, R8: footprint Resistor_THT:R_Axial_DIN0207_L6.3mm_D2.5mm_P7.62mm_Horizontal -> Resistor_SMD:R_0603_1608Metric_Pad0.98x0.95mm_HandSolder
Connections:
- net 0: now also R4.1, J1.2 (Pin_2), RV1.2
- net 3.3V: now also J1.1 (Pin_1)
- net V_out: now also J1.4 (Pin_4)
- net at R1.1, U3.3 (+): now also J2.1 (Pin_1)
- net at U2.6 (-): now also R4.2, J3.1 (Pin_1); no longer R4.1
- net at R5.1, U2.7: now also RV2.3; no longer R4.2
- net V_IN: now reaches U2.3 (+)
- net V_IN: now also J1.3 (Pin_3)
- new net: J3.2 (Pin_2), RV2.2
- new net: J2.2 (Pin_2), RV1.3
- no-connect marks 0 -> 2
Other:
- moved on the sheet: R1, R4, U3A

Commit message: V3
Parts:
- added R2, R3: R, Resistor_THT:R_Axial_DIN0207_L6.3mm_D2.5mm_P7.62mm_Horizontal, symbol Device:R
- added U1: LM35-LP, Package_TO_SOT_THT:TO-92_Inline, symbol Sensor_Temperature:LM35-LP
Connections:
- net 0: now also U1.3 (GND)
- net 3.3V: now also U1.1 (+V_{S})
- net V_IN: no longer names the net of U2.3 (+)
- net V_IN: now also R2.1, U1.2 (V_{OUT}); no longer J1.3 (Pin_3)
- new net: R2.2, R3.1
- new net V_3.3: J1.3 (Pin_3), R3.2
Other:
- moved on the sheet: J1

Commit message: final
Parts:
- removed R1: R, Resistor_SMD:R_0603_1608Metric_Pad0.98x0.95mm_HandSolder, symbol Device:R
- added J4: Conn_01x02_Pin, Connector_PinHeader_2.54mm:PinHeader_1x02_P2.54mm_Vertical, symbol Connector:Conn_01x02_Pin
- J1: footprint Connector_PinHeader_2.54mm:PinHeader_1x04_P2.54mm_Vertical -> Connector_PinSocket_2.54mm:PinSocket_1x04_P2.54mm_Vertical
- U2, U3: footprint (none) -> Package_DIP:DIP-8_W7.62mm
Connections:
- net 0: now also J1.1 (Pin_1), RV1.3, J4.2 (Pin_2); no longer J1.2 (Pin_2), RV1.2
- net 3.3V: now also J1.3 (Pin_3), RV1.1; no longer J1.1 (Pin_1), U2.8 (V+), U3.8 (V+)
- net V_3.3: now also J1.4 (Pin_4); no longer J1.3 (Pin_3)
- net V_out: now also J1.2 (Pin_2); no longer J1.4 (Pin_4)
- net at RV2.1: now also R5.1, U2.7
- net at J2.2 (Pin_2): now also U3.3 (+); no longer RV1.3
- net at J2.1 (Pin_1): now also RV1.2; no longer U3.3 (+)
- net V_ADC: now reaches U2.1, U2.2 (-), U2.5 (+)
- new net 9V: J4.1 (Pin_1), U2.8 (V+), U3.8 (V+)
- now unconnected: RV2.3
- no-connect marks 2 -> 1
Other:
- moved on the sheet: J2, J3, R2, R3, R4, R5, R6, R7, R8, RV1, RV2, U1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
